Commit message: working arm again

File: ur5_RL/envs/urdf/real_arm.urdf (robot description, URDF)
Before this commit: robot sisbot, 11 links, 10 joints
Links:
- link right_gripper: geometry collision box size=0.02 0.02 0.15; visual mesh filename=../meshes/ur5/visual/l_gripper_tip_scaled.stl scale=1 1 1
Joints:
- joint left_gripper_motor: origin xyz=-0.05 0.1 0.00 rpy=-1.57 0.0 0.0 -> xyz=-0.05 0.1 0.005 rpy=-1.57 0.0 0.0
- joint right_gripper_motor: origin xyz=0.05 0.1 0.000 rpy=-1.57 0.0 0.0 -> xyz=0.05 0.1 -0.005 rpy=-1.57 0.0 0.0

Commit message: #

File: ur5_RL/envs/urdf/real_arm.urdf (robot description, URDF)
Before this commit: robot sisbot, 11 links, 10 joints
Links:
- link right_gripper: geometry collision box size=0.025 0.02 0.15; visual mesh filename=../meshes/ur5/visual/l_gripper_tip_scaled.stl scale=1 1 1

Commit message: gripping even better

File: ur5_RL/envs/urdf/real_arm.urdf (robot description, URDF)
Before this commit: robot sisbot, 11 links, 10 joints
Joints:
- joint left_gripper_motor: limit lower=-0.00 upper=0.04 effort=300.0 velocity=100 -> lower=-0.00 upper=0.04 effort=10.0 velocity=100
- joint right_gripper_motor: limit lower=-0.04 upper=0.0 effort=300.0 velocity=100 -> lower=-0.04 upper=0.0 effort=10.0 velocity=100
